File: PCB_WORKSHOP_MUDS_MARS.kicad_sch (KiCad schematic)
At the start: 38 parts, among them J1 Conn_01x02_Pin, J2 Conn_01x02_Pin, J3 Conn_01x15_Socket, J4 Conn_01x15_Socket, J5 Conn_01x15_Socket, J6 Conn_01x02_Pin, M1 SI2300, SW1 SW_Push, U1 L9110S

Commit message: Silk screen adjustments
Parts:
- renumbered J2 to J1, J6 to J2, J1 to J3, J3 to J4, J4 to J5, J5 to J6, M1 to U2
Changed lines of the file:
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@@
 		(on_board yes)
 		(dnp no)
-		(property "Reference" "J4"
+		(property "Reference" "J5"
 			(at 177.292 13.462 0)
 			(effects
@@
 			(project "PCB_WORKSHOP_MUDS_MARS"
 				(path "/4d11e860-8407-4713-b75d-b6b01b4fa32a"
-					(reference "J4")
+					(reference "J5")
 					(unit 1)
 				)
@@
 		(dnp no)
 		(fields_autoplaced yes)
-		(property "Reference" "J2"
+		(property "Reference" "J1"
 			(at 39.37 168.2749 90)
 			(effects
@@
 			(project "PCB_WORKSHOP_MUDS_MARS"
 				(path "/4d11e860-8407-4713-b75d-b6b01b4fa32a"
-					(reference "J2")
+					(reference "J1")
 					(unit 1)
 				)
@@
 		(dnp no)
 		(fields_autoplaced yes)
-		(property "Reference" "J6"
+		(property "Reference" "J2"
 			(at 129.54 160.6549 90)
 			(effects
@@
 			(project "PCB_WORKSHOP_MUDS_MARS"
 				(path "/4d11e860-8407-4713-b75d-b6b01b4fa32a"
-					(reference "J6")
+					(reference "J2")
 					(unit 1)
 				)
@@
 		(dnp no)
 		(fields_autoplaced yes)
-		(property "Reference" "J1"
+		(property "Reference" "J3"
 			(at 73.66 22.2249 90)
 			(effects
@@
 			(project ""
 				(path "/4d11e860-8407-4713-b75d-b6b01b4fa32a"
-					(reference "J1")
+					(reference "J3")
 					(unit 1)
 				)
@@
 		(on_board yes)
 		(dnp no)
-		(property "Reference" "J3"
+		(property "Reference" "J4"
 			(at 143.002 13.462 0)
 			(effects
@@
 			(project ""
 				(path "/4d11e860-8407-4713-b75d-b6b01b4fa32a"
-					(reference "J3")
+					(reference "J4")
 					(unit 1)
 				)
@@
 		(on_board yes)
 		(dnp no)
-		(property "Reference" "J5"
+		(property "Reference" "J6"
 			(at 196.342 13.462 0)
 			(effects
@@
 			(project "PCB_WORKSHOP_MUDS_MARS"
 				(path "/4d11e860-8407-4713-b75d-b6b01b4fa32a"
-					(reference "J5")
+					(reference "J6")
 					(unit 1)
 				)
@@
 		(dnp no)
 		(fields_autoplaced yes)
-		(property "Reference" "M1"
+		(property "Reference" "U2"
 			(at 71.12 65.6937 90)
 			(effects
@@
 			(project ""
 				(path "/4d11e860-8407-4713-b75d-b6b01b4fa32a"
-					(reference "M1")
-					(unit 1)
-				)
+					(reference "U2")
+					(unit 1)
+				)
